File: MicroFlux/MicroFlux.kicad_pcb (KiCad board)
At the start: 2 copper layers, 30.5 x 53.3 mm, 24 parts, among them J1 Audio Out, J2 Audio In, U1 LM358

Commit message: restructured directories
Routing:
- added copper zone on B.Cu, net GNDREF
- removed copper zone on B.Cu, net (none)
Changed lines of the file:
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@@
     (solder_mask_min_width 0.25)
     (aux_axis_origin 0 0)
-    (visible_elements FFFFFF7F)
+    (visible_elements FFFFFFFF)
     (pcbplotparams
-      (layerselection 0x010fc_ffffffff)
+      (layerselection 0x310fc_ffffffff)
       (usegerberextensions false)
       (usegerberattributes false)
@@
       (outputformat 1)
       (mirror false)
-      (drillshape 1)
+      (drillshape 0)
       (scaleselection 1)
-      (outputdirectory ""))
+      (outputdirectory "../grb/"))
   )
   (net 0 "")
@@
     (descr https://eu.mouser.com/datasheet/2/209/EPD-200766-1274481.pdf)
     (tags "9V Battery Holder")
-    (fp_text reference BT1 (at -2.95 -6.35) (layer B.SilkS)
+    (fp_text reference BT1 (at 0 -6.35) (layer B.SilkS)
       (effects (font (size 1 1) (thickness 0.15)) (justify mirror))
     )
@@
     (polygon
       (pts
-        (xy 167.64 62.23) (xy 200.66 62.23) (xy 200.66 118.11) (xy 167.64 118.11)
+        (xy 167.64 60.96) (xy 200.66 60.96) (xy 200.66 119.38) (xy 167.64 119.38)
       )
     )
   )
-  (zone (net 0) (net_name "") (layer B.Cu) (hatch edge 0.508)
+  (zone (net 2) (net_name GNDREF) (layer B.Cu) (hatch edge 0.508)
     (connect_pads (clearance 0.508))
     (min_thickness 0.254)
@@
     (polygon
       (pts
-        (xy 166.37 60.96) (xy 201.93 60.96) (xy 201.93 119.38) (xy 166.37 119.38)
+        (xy 166.37 62.23) (xy 201.93 62.23) (xy 201.93 118.11) (xy 166.37 118.11)
       )
     )

Commit message: added logos on board
Parts:
- added REF**: KiCAD Logo, Symbol:Symbol_KiCAD-Logo_CopperAndSilkScreenTop, B.Cu at (195.6, 71.1)
- added REF**: OSHW-Logo2_7.3x6mm_Copper, Symbol:OSHW-Logo2_7.3x6mm_Copper, F.Cu at (172.7, 113.0)

Commit message: assigned MPNs
Parts:
- C3, C4: value C -> 10u
- C5, C6: value C -> 100n
- C7, C8: value CP -> 10u; footprint Capacitor_THT:CP_Radial_D5.0mm_P2.50mm -> Capacitor_THT:C_Disc_D3.0mm_W1.6mm_P2.50mm
- D1: value LED -> green
- D2: value D_Schottky -> 1N5818-T; footprint Diode_THT:D_DO-34_SOD68_P7.62mm_Horizontal -> Diode_THT:D_DO-41_SOD81_P7.62mm_Horizontal
- R5, R6, R7: value R -> 1k
- RV1: value Alps_RK097 -> 10k
- moved C7 1.27 mm to (177.8, 87.7)
- moved C8 1.27 mm to (190.5, 90.2)
- moved REF** 0.63 mm to (196.2, 71.1), turned to 90 degrees
Routing:
- net Net-(C4-Pad1): track 20.1 -> 17.9 mm
- net Net-(C3-Pad1): track 20.1 -> 18.2 mm

Commit message: added version information and locked logos on board
Parts:
- U1: value LM358 -> AS358P-E1
- moved REF** 0.63 mm to (195.6, 71.1), turned to 270 degrees
- moved REF** 0.63 mm to (172.1, 113.0), turned to 90 degrees
Other:
- board text added: "MicroFlux"
- board text added: "github.com/FOSHSolderKits"
- board text added: "v0.1"
